Commit message: Update Basler_ace2_GigE.urdf

File: Blaser_AG/ACE2/urdf/Basler_ace2_GigE.urdf (robot description, URDF)
Before this commit: robot basler_camera, 1 links, 0 joints
Links:
- link camera: geometry collision mesh filename=package://ACE2/meshes/Basler_ace2_GigE.stl scale=0.001 0.001 0.001; visual mesh filename=package://ACE2/meshes/Basler_ace2_GigE.stl scale=0.001 0.001 0.001
