Commit message: Update logitech_c920_web_cam_cover.urdf

File: logitech/c920/urdf/logitech_c920_web_cam_cover.urdf (robot description, URDF)
Before this commit: robot logitech_c920_web_cam_cover, 1 links, 0 joints
Links:
- link cover_link: geometry collision mesh filename=package://c920/meshes/Logitech_C920_Web_Cam_Cover.stl scale=0.001 0.001 0.001; visual mesh filename=package://c920/meshes/Logitech_C920_Web_Cam_Cover.stl scale=0.001 0.001 0.001
