Commit message: Update logitech-c920.urdf

File: logitech/c920/urdf/logitech-c920.urdf (robot description, URDF)
Before this commit: robot untitled_model, 1 links, 1 joints
Links:
- link model_link: geometry collision mesh filename=package://c920/meshes/logitech-c920.stl; visual mesh filename=package://c920/meshes/logitech-c920.stl
