Commit message: Update logitech_c920.urdf

File: logitech/c920/urdf/logitech_c920.urdf (robot description, URDF)
Before this commit: robot logitech_c920, 1 links, 0 joints
Links:
- link camera_link: geometry collision mesh filename=package://c920/meshes/logitech-c920.stl scale=0.001 0.001 0.001; visual mesh filename=package://c920/meshes/logitech-c920.stl scale=0.001 0.001 0.001

Commit message: Update logitech_c920.urdf

File: logitech/c920/urdf/logitech_c920.urdf (robot description, URDF)
Before this commit: robot logitech_c920, 1 links, 1 joints
Links:
- link camera_link: geometry collision mesh filename=package://c920/meshes/logitech-c920.stl; visual mesh filename=package://c920/meshes/logitech-c920.stl

Commit message: Update logitech_c920.urdf

File: logitech/c920/urdf/logitech_c920.urdf (robot description, URDF)
Before this commit: robot logitech_c920, 1 links, 1 joints
Links:
- removed link camera_link
- added link realsense_d455_link, mass 0.2; collision mesh filename=package://c920/meshes/logitech-c920.stl scale=0.001 0.001 0.001; visual mesh filename=package://c920/meshes/logitech-c920.stl scale=0.001 0.001 0.001
Joints:
- removed joint world_to_camera

Commit message: Update logitech_c920.urdf

File: logitech/c920/urdf/logitech_c920.urdf (robot description, URDF)
Before this commit: robot logitech_c920, 1 links, 0 joints
Links:
- link camera: geometry collision mesh filename=package://c920/meshes/logitech_c920.stl scale=1 1 1; visual mesh filename=package://c920/meshes/logitech_c920.stl scale=1 1 1

Commit message: Update logitech_c920.urdf

File: logitech/c920/urdf/logitech_c920.urdf (robot description, URDF)
Before this commit: robot logitech_c920, 1 links, 0 joints
Links:
- link logitech_c920_link: geometry collision mesh filename=package://c920/meshes/logitech_c920.stl scale=0.01 0.01 0.01; visual mesh filename=package://c920/meshes/logitech_c920.stl scale=0.01 0.01 0.01

Commit message: Update logitech_c920.urdf

File: logitech/c920/urdf/logitech_c920.urdf (robot description, URDF)
Before this commit: robot logitech_c920, 1 links, 0 joints
Links:
- link camera_link: geometry collision mesh filename=package://c920/meshes/logitech_c920.stl scale=1 1 1; visual mesh filename=package://c920/meshes/logitech_c920.stl scale=1 1 1

Commit message: Update logitech_c920.urdf

File: logitech/c920/urdf/logitech_c920.urdf (robot description, URDF)
Before this commit: robot logitech_c920, 1 links, 0 joints
Links:
- link logitech_c920_link: geometry collision mesh filename=package://c920/meshes/logitech_920.stl scale=1 1 1; visual mesh filename=package://c920/meshes/logitech_920.stl scale=1 1 1

Commit message: Update logitech_c920.urdf

File: logitech/c920/urdf/logitech_c920.urdf (robot description, URDF)
Before this commit: robot logitech_c920, 1 links, 0 joints
Links:
- link logitech_c920_link: geometry collision mesh filename=package://c920/meshes/logitech_920.stl scale=-1000 -1000 -1000; visual mesh filename=package://c920/meshes/logitech_920.stl scale=-1000 -1000 -1000

Commit message: Update logitech_c920.urdf

File: logitech/c920/urdf/logitech_c920.urdf (robot description, URDF)
Before this commit: robot logitech_c920, 1 links, 0 joints
Links:
- link logitech_c920_link: mass 0.162 -> 0

Commit message: changed the urdf and stl for the logitech c920

File: logitech/c920/urdf/logitech_c920.urdf (robot description, URDF)
Before this commit: robot logitech_c920, 1 links, 0 joints
Links:
- link logitech_c920_link: geometry collision mesh filename=package://c920/meshes/Logitech_C920_.stl scale=0.001 0.001 0.001; visual mesh filename=package://c920/meshes/Logitech_C920_.stl scale=0.001 0.001 0.001

Commit message: Update logitech_c920.urdf

File: logitech/c920/urdf/logitech_c920.urdf (robot description, URDF)
Before this commit: robot logitech_c920, 1 links, 0 joints
Links:
- link logitech_c920_link: mass 0 -> 0.162

Commit message: c920 upload

File: logitech/c920/urdf/logitech_c920.urdf (robot description, URDF)
Before this commit: robot logitech_c920, 1 links, 0 joints
Links:
- link logitech_c920_link: geometry collision mesh filename=package://c920/meshes/Logi_920.stl scale=0.001 0.001 0.001; visual mesh filename=package://c920/meshes/Logi_920.stl scale=0.001 0.001 0.001

Commit message: Update logitech_c920.urdf

File: logitech/c920/urdf/logitech_c920.urdf (robot description, URDF)
Before this commit: robot logitech_c920, 1 links, 0 joints
Links:
- link logitech_c920_link: geometry collision mesh filename=package://c920/meshes/Logi_920.stl; visual mesh filename=package://c920/meshes/Logi_920.stl
