Commit message: Update Pi_Camerav3.urdf

File: Raspberry/Pi_CameraV3/urdf/Pi_Camerav3.urdf (robot description, URDF)
Before this commit: robot pi_camerav3, 1 links, 0 joints
Links:
- link pi_camerav3_link: geometry collision mesh filename=package://Pi_CameraV3/meshes/Pi_CameraV3.stl scale=0.001 0.001 0.001; visual mesh filename=package://Pi_CameraV3/meshes/Pi_CameraV3.stl scale=0.001 0.001 0.001
