Commit message: Update gen1_0.urdf

File: Generic Cameras/Gen1_0/urdf/gen1_0.urdf (robot description, URDF)
Before this commit: robot gen1_0, 1 links, 0 joints
Links:
- link gen1_0_link: geometry collision mesh filename=package://Gen1_0/meshes/gen1_0.stl scale=0.001 0.001 0.001; visual mesh filename=package://Gen1_0/meshes/gen1_0.stl scale=0.001 0.001 0.001
