Commit message: sizes changed for gen11

File: Generic_Cameras/Gen1_0/urdf/Gen_11cyb.urdf (robot description, URDF)
Before this commit: robot gen1_0, 1 links, 0 joints
Links:
- link gen1_0_link: mass 0.05 -> 0.1; geometry collision mesh filename=package://Gen1_0/meshes/Gen_11cyb.stl scale=0.001 0.001 0.001; visual mesh filename=package://Gen1_0/meshes/Gen_11cyb.stl scale=0.001 0.001 0.001
