Commit message: new generic camera mesh and urdf

File: Generic_Cameras/Gen1_0/urdf/Generic11.urdf (robot description, URDF)
Before this commit: robot gen1_0, 1 links, 0 joints
Links:
- removed link gen1_0_link
- added link generic_camera_link, mass 0.1; collision mesh filename=package://Gen1_0/meshes/Generic11.stl scale=0.001 0.001 0.001; visual mesh filename=package://Gen1_0/meshes/Generic11.stl scale=0.001 0.001 0.001
