Commit message: IP camera resized

File: Generic_Cameras/Generic_IP_camera/urdf/IPCamera2.urdf (robot description, URDF)
Before this commit: robot generic_ip_cam, 1 links, 0 joints
Links:
- removed link generic_ip_cam_link
- added link generic_ip_camera_link, mass 0.15; collision mesh filename=package://Generic_IP_camera/meshes/IPCamera2.stl scale=0.001 0.001 0.001; visual mesh filename=package://Generic_IP_camera/meshes/IPCamera2.stl scale=0.001 0.001 0.001
