Commit message: IPcamera rotation

File: Generic_Cameras/Generic_IP_camera/urdf/IPCamera21.urdf (robot description, URDF)
Before this commit: robot generic_ip_camera, 1 links, 0 joints
Links:
- removed link generic_ip_camera_link
- added link ip_camera_link, mass 0.15; collision mesh filename=package://Generic_IP_camera/meshes/IPCamera21.stl scale=0.001 0.001 0.001; visual mesh filename=package://Generic_IP_camera/meshes/IPCamera21.stl scale=0.001 0.001 0.001
