Commit message: NVR change1

File: Generic_Cameras/Generic_NVR/urdf/NVRGeneric.urdf (robot description, URDF)
Before this commit: robot nvr_generic, 1 links, 0 joints
Links:
- link nvr_generic_link: geometry collision mesh filename=package://Generic_NVR/meshes/NVRGeneric.stl scale=0.001 0.001 0.001; visual mesh filename=package://Generic_NVR/meshes/NVRGeneric.stl scale=0.001 0.001 0.001
