Commit message: updating NVR

File: Generic_Cameras/Generic_NVR/urdf/GenericNVR.urdf (robot description, URDF)
Before this commit: robot nvr_generic, 1 links, 0 joints
Links:
- removed link nvr_generic_link
- added link nvr_link, mass 1.5; collision mesh filename=package://Generic_NVR/meshes/GenericNVR.stl scale=0.001 0.001 0.001; visual mesh filename=package://Generic_NVR/meshes/GenericNVR.stl scale=0.001 0.001 0.001
