Commit message: NVR_update

File: Generic_Cameras/Generic_NVR/urdf/GenericNVR2.urdf (robot description, URDF)
Before this commit: robot generic_nvr, 1 links, 0 joints
Links:
- removed link nvr_link
- added link generic_nvr_link, mass 0.5; collision mesh filename=package://Generic_NVR/meshes/GenericNVR2.stl scale=0.001 0.001 0.001; visual mesh filename=package://Generic_NVR/meshes/GenericNVR2.stl scale=0.001 0.001 0.001
