Commit message: folder renamed

File: KUKA_LBR/iiwa14_r820/urdf/iiwa14.xacro (robot description, xacro)
@@ -2,9 +2,9 @@
 <robot xmlns:xacro="http://www.ros.org/wiki/xacro">
   <!-- Import all Gazebo-customization elements, including Gazebo colors -->
-  <xacro:include filename="$(find iiwa14 r820)/urdf/iiwa.gazebo.xacro" />
+  <xacro:include filename="$(find iiwa14_r820)/urdf/iiwa.gazebo.xacro" />
   <!-- Import Transmissions -->
-  <xacro:include filename="$(find iiwa14 r820)/urdf/iiwa.transmission.xacro" />
+  <xacro:include filename="$(find iiwa14_r820)/urdf/iiwa.transmission.xacro" />
   <!-- Include Utilities -->
-  <xacro:include filename="$(find iiwa14 r820)/urdf/utilities.xacro" />
+  <xacro:include filename="$(find iiwa14_r820)/urdf/utilities.xacro" />
   <!-- some constants -->
   <xacro:property name="safety_controller_k_pos" value="100" />
@@ -44,5 +44,5 @@
         <origin xyz="0 0 0" rpy="0 0 0"/>
         <geometry>
-          <mesh filename="package://iiwa14 r820/meshes/iiwa14/visual/link_0.stl"/>
+          <mesh filename="package://iiwa14_r820/meshes/iiwa14/visual/link_0.stl"/>
         </geometry>
         <material name="Grey"/>
@@ -51,5 +51,5 @@
         <origin xyz="0 0 0" rpy="0 0 0"/>
         <geometry>
-          <mesh filename="package://iiwa14 r820/meshes/iiwa14/collision/link_0_s.stl"/>
+          <mesh filename="package://iiwa14_r820/meshes/iiwa14/collision/link_0_s.stl"/>
         </geometry>
         <material name="Grey"/>
@@ -85,12 +85,12 @@
         <origin xyz="0 0 0" rpy="0 0 0"/>
         <geometry>
-          <mesh filename="package://iiwa14 r820/meshes/iiwa14/visual/link_1.stl"/>
-        </geometry>
-        <material name="Orange"/>
-      </visual>
-      <collision>
-        <origin xyz="0 0 0" rpy="0 0 0"/>
-        <geometry>
-          <mesh filename="package://iiwa14 r820/meshes/iiwa14/collision/link_1_s.stl"/>
+          <mesh filename="package://iiwa14_r820/meshes/iiwa14/visual/link_1.stl"/>
+        </geometry>
+        <material name="Orange"/>
+      </visual>
+      <collision>
+        <origin xyz="0 0 0" rpy="0 0 0"/>
+        <geometry>
+          <mesh filename="package://iiwa14_r820/meshes/iiwa14/collision/link_1_s.stl"/>
         </geometry>
         <material name="Orange"/>
@@ -120,12 +120,12 @@
         <origin xyz="0 0 0" rpy="0 0 0"/>
         <geometry>
-          <mesh filename="package://iiwa14 r820/meshes/iiwa14/visual/link_2.stl"/>
-        </geometry>
-        <material name="Orange"/>
-      </visual>
-      <collision>
-        <origin xyz="0 0 0" rpy="0 0 0"/>
-        <geometry>
-          <mesh filename="package://iiwa14 r820/meshes/iiwa14/collision/link_2_s.stl"/>
+          <mesh filename="package://iiwa14_r820/meshes/iiwa14/visual/link_2.stl"/>
+        </geometry>
+        <material name="Orange"/>
+      </visual>
+      <collision>
+        <origin xyz="0 0 0" rpy="0 0 0"/>
+        <geometry>
+          <mesh filename="package://iiwa14_r820/meshes/iiwa14/collision/link_2_s.stl"/>
         </geometry>
         <material name="Orange"/>
@@ -155,12 +155,12 @@
         <origin xyz="0 0 0" rpy="0 0 0"/>
         <geometry>
-          <mesh filename="package://iiwa14 r820/meshes/iiwa14/visual/link_3.stl"/>
-        </geometry>
-        <material name="Orange"/>
-      </visual>
-      <collision>
-        <origin xyz="0 0 0" rpy="0 0 0"/>
-        <geometry>
-          <mesh filename="package://iiwa14 r820/meshes/iiwa14/collision/link_3_s.stl"/>
+          <mesh filename="package://iiwa14_r820/meshes/iiwa14/visual/link_3.stl"/>
+        </geometry>
+        <material name="Orange"/>
+      </visual>
+      <collision>
+        <origin xyz="0 0 0" rpy="0 0 0"/>
+        <geometry>
+          <mesh filename="package://iiwa14_r820/meshes/iiwa14/collision/link_3_s.stl"/>
         </geometry>
         <material name="Orange"/>
@@ -190,12 +190,12 @@
         <origin xyz="0 0 0" rpy="0 0 0"/>
         <geometry>
-          <mesh filename="package://iiwa14 r820/meshes/iiwa14/visual/link_4.stl"/>
-        </geometry>
-        <material name="Orange"/>
-      </visual>
-      <collision>
-        <origin xyz="0 0 0" rpy="0 0 0"/>
-        <geometry>
-          <mesh filename="package://iiwa14 r820/meshes/iiwa14/collision/link_4_s.stl"/>
+          <mesh filename="package://iiwa14_r820/meshes/iiwa14/visual/link_4.stl"/>
+        </geometry>
+        <material name="Orange"/>
+      </visual>
+      <collision>
+        <origin xyz="0 0 0" rpy="0 0 0"/>
+        <geometry>
+          <mesh filename="package://iiwa14_r820/meshes/iiwa14/collision/link_4_s.stl"/>
         </geometry>
         <material name="Orange"/>
@@ -225,12 +225,12 @@
         <origin xyz="0 0 0" rpy="0 0 0"/>
         <geometry>
-          <mesh filename="package://iiwa14 r820/meshes/iiwa14/visual/link_5.stl"/>
-        </geometry>
-        <material name="Orange"/>
-      </visual>
-      <collision>
-        <origin xyz="0 0 0" rpy="0 0 0"/>
-        <geometry>
-          <mesh filename="package://iiwa14 r820/meshes/iiwa14/collision/link_5_s.stl"/>
+          <mesh filename="package://iiwa14_r820/meshes/iiwa14/visual/link_5.stl"/>
+        </geometry>
+        <material name="Orange"/>
+      </visual>
+      <collision>
+        <origin xyz="0 0 0" rpy="0 0 0"/>
+        <geometry>
+          <mesh filename="package://iiwa14_r820/meshes/iiwa14/collision/link_5_s.stl"/>
         </geometry>
         <material name="Orange"/>
@@ -260,12 +260,12 @@
         <origin xyz="0 0 0" rpy="0 0 0"/>
         <geometry>
-          <mesh filename="package://iiwa14 r820/meshes/iiwa14/visual/link_6.stl"/>
-        </geometry>
-        <material name="Orange"/>
-      </visual>
-      <collision>
-        <origin xyz="0 0 0" rpy="0 0 0"/>
-        <geometry>
-          <mesh filename="package://iiwa14 r820/meshes/iiwa14/collision/link_6_s.stl"/>
+          <mesh filename="package://iiwa14_r820/meshes/iiwa14/visual/link_6.stl"/>
+        </geometry>
+        <material name="Orange"/>
+      </visual>
+      <collision>
+        <origin xyz="0 0 0" rpy="0 0 0"/>
+        <geometry>
+          <mesh filename="package://iiwa14_r820/meshes/iiwa14/collision/link_6_s.stl"/>
         </geometry>
         <material name="Orange"/>
@@ -295,6 +295,6 @@
         <origin xyz="0 0 0" rpy="0 0 0"/>
         <geometry>
-<!--           <mesh filename="package://iiwa14 r820/meshes/iiwa14/visual/link_7.stl"/> -->
-		  <mesh filename="package://iiwa14 r820/meshes/iiwa14/visual/link_7-MF-Touch-pneumatisch.stl"/>
+<!--           <mesh filename="package://iiwa14_r820/meshes/iiwa14/visual/link_7.stl"/> -->
+		  <mesh filename="package://iiwa14_r820/meshes/iiwa14/visual/link_7-MF-Touch-pneumatisch.stl"/>
         </geometry>
         <material name="Grey"/>
@@ -303,6 +303,6 @@
         <origin xyz="0 0 0" rpy="0 0 0"/>
         <geometry>
-<!--           <mesh filename="package://iiwa14 r820/meshes/iiwa14/collision/link_7_s.stl"/> -->
-		  <mesh filename="package://iiwa14 r820/meshes/iiwa14/collision/link_7-MF-Touch-pneumatisch_s.stl"/>
+<!--           <mesh filename="package://iiwa14_r820/meshes/iiwa14/collision/link_7_s.stl"/> -->
+		  <mesh filename="package://iiwa14_r820/meshes/iiwa14/collision/link_7-MF-Touch-pneumatisch_s.stl"/>
         </geometry>
         <material name="Grey"/>
