Commit message: Z1 reupload

File: Unitree/z1_description/xacro/z1.urdf (robot description, URDF)
Before this commit: robot z1_description, 8 links, 7 joints
Links:
- link link00: geometry collision cylinder length=0.051 radius=0.0325; visual mesh filename=package://z1_description/meshes/visual/z1_Link00.stl scale=1 1 1
- link link01: geometry visual mesh filename=package://z1_description/meshes/visual/z1_Link01.stl scale=1 1 1
- link link02: geometry collision cylinder length=0.051 radius=0.0325; collision cylinder length=0.102 radius=0.0325
- link link03: geometry collision cylinder length=0.059 radius=0.0325; collision cylinder length=0.116 radius=0.02
- link link04: geometry collision cylinder length=0.067 radius=0.0325; visual mesh filename=package://z1_description/meshes/visual/z1_Link04.stl scale=1 1 1
- link link05: geometry visual mesh filename=package://z1_description/meshes/visual/z1_Link05.stl scale=1 1 1
- link link06: geometry collision cylinder length=0.051 radius=0.0325; visual mesh filename=package://z1_description/meshes/visual/z1_Link06.stl scale=1 1 1
