Commit message: H1 fix

File: Unitree/h1_description/urdf/h1_with_hand.urdf (robot description, URDF)
Before this commit: robot H1/, 52 links, 51 joints
Links:
- link L_hand_base_link: geometry collision mesh filename=package://h1_description/meshes/L_hand_base_link.STL; visual mesh filename=package://h1_description/meshes/L_hand_base_link.stl
- link L_index_intermediate: geometry collision mesh filename=package://h1_description/meshes/Link16_L.STL; visual mesh filename=package://h1_description/meshes/Link16_L.stl
- link L_index_proximal: geometry collision mesh filename=package://h1_description/meshes/Link15_L.STL; visual mesh filename=package://h1_description/meshes/Link15_L.stl
- link L_middle_intermediate: geometry collision mesh filename=package://h1_description/meshes/Link18_L.STL; visual mesh filename=package://h1_description/meshes/Link18_L.stl
- link L_middle_proximal: geometry collision mesh filename=package://h1_description/meshes/Link17_L.STL; visual mesh filename=package://h1_description/meshes/Link17_L.stl
- link L_pinky_intermediate: geometry collision mesh filename=package://h1_description/meshes/Link22_L.STL; visual mesh filename=package://h1_description/meshes/Link22_L.stl
- link L_pinky_proximal: geometry collision mesh filename=package://h1_description/meshes/Link21_L.STL; visual mesh filename=package://h1_description/meshes/Link21_L.stl
- link L_ring_intermediate: geometry collision mesh filename=package://h1_description/meshes/Link20_L.STL; visual mesh filename=package://h1_description/meshes/Link20_L.stl
- link L_ring_proximal: geometry collision mesh filename=package://h1_description/meshes/Link19_L.STL; visual mesh filename=package://h1_description/meshes/Link19_L.stl
- link L_thumb_distal: geometry collision mesh filename=package://h1_description/meshes/Link14_L.STL; visual mesh filename=package://h1_description/meshes/Link14_L.stl
- link L_thumb_intermediate: geometry collision mesh filename=package://h1_description/meshes/Link13_L.STL; visual mesh filename=package://h1_description/meshes/Link13_L.stl
- link L_thumb_proximal: geometry collision mesh filename=package://h1_description/meshes/Link12_L.STL; visual mesh filename=package://h1_description/meshes/Link12_L.stl
- link L_thumb_proximal_base: geometry collision mesh filename=package://h1_description/meshes/Link11_L.STL; visual mesh filename=package://h1_description/meshes/Link11_L.stl
- link R_hand_base_link: geometry collision mesh filename=package://h1_description/meshes/R_hand_base_link.STL; visual mesh filename=package://h1_description/meshes/R_hand_base_link.stl
- link R_index_intermediate: geometry collision mesh filename=package://h1_description/meshes/Link16_R.STL; visual mesh filename=package://h1_description/meshes/Link16_R.stl
- link R_index_proximal: geometry collision mesh filename=package://h1_description/meshes/Link15_R.STL; visual mesh filename=package://h1_description/meshes/Link15_R.stl
- link R_middle_intermediate: geometry collision mesh filename=package://h1_description/meshes/Link18_R.STL; visual mesh filename=package://h1_description/meshes/Link18_R.stl
- link R_middle_proximal: geometry collision mesh filename=package://h1_description/meshes/Link17_R.STL; visual mesh filename=package://h1_description/meshes/Link17_R.stl
- link R_pinky_intermediate: geometry collision mesh filename=package://h1_description/meshes/Link22_R.STL; visual mesh filename=package://h1_description/meshes/Link22_R.stl
- link R_pinky_proximal: geometry collision mesh filename=package://h1_description/meshes/Link21_R.STL; visual mesh filename=package://h1_description/meshes/Link21_R.stl
- link R_ring_intermediate: geometry collision mesh filename=package://h1_description/meshes/Link20_R.STL; visual mesh filename=package://h1_description/meshes/Link20_R.stl
- link R_ring_proximal: geometry collision mesh filename=package://h1_description/meshes/Link19_R.STL; visual mesh filename=package://h1_description/meshes/Link19_R.stl
- link R_thumb_distal: geometry collision mesh filename=package://h1_description/meshes/Link14_R.STL; visual mesh filename=package://h1_description/meshes/Link14_R.stl
- link R_thumb_intermediate: geometry collision mesh filename=package://h1_description/meshes/Link13_R.STL; visual mesh filename=package://h1_description/meshes/Link13_R.stl
- link R_thumb_proximal: geometry collision mesh filename=package://h1_description/meshes/Link12_R.STL; visual mesh filename=package://h1_description/meshes/Link12_R.stl
- link R_thumb_proximal_base: geometry collision mesh filename=package://h1_description/meshes/Link11_R.STL; visual mesh filename=package://h1_description/meshes/Link11_R.stl
- link left_ankle_link: geometry collision box size=0.28 0.03 0.024; visual mesh filename=package://h1_description/meshes/left_ankle_link.stl
- link left_elbow_link: geometry collision cylinder length=0.09 radius=0.03; visual mesh filename=package://h1_description/meshes/left_elbow_link.stl
- link left_hand_link: geometry collision mesh filename=package://h1_description/meshes/left_hand_link.STL; visual mesh filename=package://h1_description/meshes/left_hand_link.stl
- link left_hip_pitch_link: geometry collision cylinder length=0.2 radius=0.05; visual mesh filename=package://h1_description/meshes/left_hip_pitch_link.stl
- link left_hip_roll_link: geometry collision cylinder length=0.01 radius=0.02; visual mesh filename=package://h1_description/meshes/left_hip_roll_link.stl
- link left_hip_yaw_link: geometry collision cylinder length=0.02 radius=0.01; visual mesh filename=package://h1_description/meshes/left_hip_yaw_link.stl
- link left_knee_link: geometry collision cylinder length=0.2 radius=0.05; visual mesh filename=package://h1_description/meshes/left_knee_link.stl
- link left_shoulder_pitch_link: geometry collision cylinder length=0.04 radius=0.03; visual mesh filename=package://h1_description/meshes/left_shoulder_pitch_link.stl
- link left_shoulder_roll_link: geometry collision cylinder length=0.01 radius=0.04; visual mesh filename=package://h1_description/meshes/left_shoulder_roll_link.stl
- link left_shoulder_yaw_link: geometry collision cylinder length=0.01 radius=0.04; visual mesh filename=package://h1_description/meshes/left_shoulder_yaw_link.stl
- link logo_link: geometry visual mesh filename=package://h1_description/meshes/logo_link.stl
- link pelvis: geometry collision sphere radius=0.05; visual mesh filename=package://h1_description/meshes/pelvis.stl
- link right_ankle_link: geometry collision box size=0.28 0.03 0.024; visual mesh filename=package://h1_description/meshes/right_ankle_link.stl
- link right_elbow_link: geometry collision cylinder length=0.09 radius=0.03; visual mesh filename=package://h1_description/meshes/right_elbow_link.stl
- link right_hand_link: geometry collision mesh filename=package://h1_description/meshes/right_hand_link.STL; visual mesh filename=package://h1_description/meshes/right_hand_link.stl
- link right_hip_pitch_link: geometry collision cylinder length=0.2 radius=0.05; visual mesh filename=package://h1_description/meshes/right_hip_pitch_link.stl
- link right_hip_roll_link: geometry collision cylinder length=0.01 radius=0.02; visual mesh filename=package://h1_description/meshes/right_hip_roll_link.stl
- link right_hip_yaw_link: geometry collision cylinder length=0.02 radius=0.01; visual mesh filename=package://h1_description/meshes/right_hip_yaw_link.stl
- link right_knee_link: geometry collision cylinder length=0.2 radius=0.05; visual mesh filename=package://h1_description/meshes/right_knee_link.stl
- link right_shoulder_pitch_link: geometry collision cylinder length=0.04 radius=0.03; visual mesh filename=package://h1_description/meshes/right_shoulder_pitch_link.s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
- link right_shoulder_roll_link: geometry collision cylinder length=0.01 radius=0.04; visual mesh filename=package://h1_description/meshes/right_shoulder_roll_link.stl
- link right_shoulder_yaw_link: geometry collision cylinder length=0.01 radius=0.04; visual mesh filename=package://h1_description/meshes/right_shoulder_yaw_link.stl
- link torso_link: geometry collision box size=0.08 0.16 0.1; visual mesh filename=package://h1_description/meshes/torso_link.stl
