Commit message: Antenna1 fix

File: Fictionlab/leo_description/urdf/leo.urdf (robot description, URDF)
Before this commit: robot leo, 12 links, 11 joints
Links:
- removed link antenna_link
- added link Antenna1_link, mass 0.001237; collision cylinder length=0.056 radius=0.0055; visual mesh filename=package://leo_description/models/Antenna1.stl
Joints:
- removed joint antenna_joint
- added joint Antenna1_joint: type fixed, parent base_link, child Antenna1_link, origin xyz=-0.0052 0.056 -0.0065 rpy=0 0 0
