Commit message: KR70_fix

File: KUKA_LBR/KR70/urdf/kr70_r2100.urdf (robot description, URDF)
Before this commit: robot kr70_r2100, 11 links, 10 joints
Links:
- link base_link: geometry collision mesh filename=package://KUKA_LBR/KR70/meshes/collision/base_link.stl; visual mesh filename=package://KUKA_LBR/KR70/meshes/visual/base_link1.stl
- link link_1: geometry collision mesh filename=package://KUKA_LBR/KR70/meshes/collision/link_1.stl; visual mesh filename=package://KUKA_LBR/KR70/meshes/visual/link_11.stl
- link link_2: geometry collision mesh filename=package://KUKA_LBR/KR70/meshes/collision/link_2.stl; visual mesh filename=package://KUKA_LBR/KR70/meshes/visual/link_21.stl
- link link_3: geometry collision mesh filename=package://KUKA_LBR/KR70/meshes/collision/link_3.stl; visual mesh filename=package://KUKA_LBR/KR70/meshes/visual/link_31.stl
- link link_4: geometry collision mesh filename=package://KUKA_LBR/KR70/meshes/collision/link_4.stl; visual mesh filename=package://KUKA_LBR/KR70/meshes/visual/link_41.stl
- link link_5: geometry collision mesh filename=package://KUKA_LBR/KR70/meshes/collision/link_5.stl; visual mesh filename=package://KUKA_LBR/KR70/meshes/visual/link_51.stl
- link link_6: geometry collision mesh filename=package://KUKA_LBR/KR70/meshes/collision/link_6.stl; visual mesh filename=package://KUKA_LBR/KR70/meshes/visual/link_61.stl

Commit message: kr70 fix2

File: KUKA_LBR/KR70/urdf/kr70_r2100.urdf (robot description, URDF)
Before this commit: robot kr70_r2100, 11 links, 10 joints
Links:
- link base_link: geometry collision mesh filename=package://KR70/meshes/collision/base_link.stl; visual mesh filename=package://KR70/meshes/visual/base_link1.stl
- link link_1: geometry collision mesh filename=package://KR70/meshes/collision/link_1.stl; visual mesh filename=package://KR70/meshes/visual/link_11.stl
- link link_2: geometry collision mesh filename=package://KR70/meshes/collision/link_2.stl; visual mesh filename=package://KR70/meshes/visual/link_21.stl
- link link_3: geometry collision mesh filename=package://KR70/meshes/collision/link_3.stl; visual mesh filename=package://KR70/meshes/visual/link_31.stl
- link link_4: geometry collision mesh filename=package://KR70/meshes/collision/link_4.stl; visual mesh filename=package://KR70/meshes/visual/link_41.stl
- link link_5: geometry collision mesh filename=package://KR70/meshes/collision/link_5.stl; visual mesh filename=package://KR70/meshes/visual/link_51.stl
- link link_6: geometry collision mesh filename=package://KR70/meshes/collision/link_6.stl; visual mesh filename=package://KR70/meshes/visual/link_61.stl

Commit message: renaming visual

File: KUKA_LBR/KR70/urdf/kr70_r2100.urdf (robot description, URDF)
Before this commit: robot kr70_r2100, 11 links, 10 joints
Links:
- link base_link: geometry collision mesh filename=package://KUKA_LBR/KR70/meshes/collision/base_link.stl; visual mesh filename=package://KUKA_LBR/KR70/meshes/visual/base_link.stl
- link link_1: geometry collision mesh filename=package://KUKA_LBR/KR70/meshes/collision/link_1.stl; visual mesh filename=package://KUKA_LBR/KR70/meshes/visual/link_1.stl
- link link_2: geometry collision mesh filename=package://KUKA_LBR/KR70/meshes/collision/link_2.stl; visual mesh filename=package://KUKA_LBR/KR70/meshes/visual/link_2.stl
- link link_3: geometry collision mesh filename=package://KUKA_LBR/KR70/meshes/collision/link_3.stl; visual mesh filename=package://KUKA_LBR/KR70/meshes/visual/link_3.stl
- link link_4: geometry collision mesh filename=package://KUKA_LBR/KR70/meshes/collision/link_4.stl; visual mesh filename=package://KUKA_LBR/KR70/meshes/visual/link_4.stl
- link link_5: geometry collision mesh filename=package://KUKA_LBR/KR70/meshes/collision/link_5.stl; visual mesh filename=package://KUKA_LBR/KR70/meshes/visual/link_5.stl
- link link_6: geometry collision mesh filename=package://KUKA_LBR/KR70/meshes/collision/link_6.stl; visual mesh filename=package://KUKA_LBR/KR70/meshes/visual/link_6.stl
