Commit message: size changed

File: Generic_Objects/Generic_Cube/urdf/default_cube.urdf (robot description, URDF)
Before this commit: robot cube_robot, 1 links, 0 joints
Links:
- link base_link: geometry collision mesh filename=package://Generic_Objects/Generic_Cube/urdf/default_cube.stl scale=1 1 1; visual mesh filename=package://Generic_Objects/Generic_Cube/urdf/default_cube.stl scale=1 1 1

Commit message: adding the mesh

File: Generic_Objects/Generic_Cube/urdf/default_cube.urdf (robot description, URDF)
Before this commit: robot cube_robot, 1 links, 0 joints
Links:
- link base_link: geometry collision mesh filename=package://Generic_Objects/Generic_Cube/meshes/default_cube.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 scale=0.01 0.01 0.01; visual mesh filename=package://Generic_Objects/Generic_Cube/meshes/default_cube.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 scale=0.01 0.01 0.01

Commit message: urdf reupload

File: Generic_Objects/Generic_Cube/urdf/default_cube.urdf (robot description, URDF)
Before this commit: robot cube_robot, 1 links, 0 joints
Links:
- removed link base_link
- added link cube_link, mass 0.1; collision mesh filename=package://Generic_Cube/meshes/default_cube.stl scale=0.001 0.001 0.001; visual mesh filename=package://Generic_Cube/meshes/default_cube.stl scale=0.001 0.001 0.001

Commit message: new cube resized

File: Generic_Objects/Generic_Cube/urdf/default_cube.urdf (robot description, URDF)
Before this commit: robot default_cube, 1 links, 0 joints
Links:
- link cube_link: mass 0.1 -> 1; geometry collision mesh filename=package://Generic_Cube/meshes/default_cube.stl scale=1 1 1; visual mesh filename=package://Generic_Cube/meshes/default_cube.stl scale=1 1 1
