Commit message: cube retry

File: Generic_Objects/Generic_Cube/urdf/recube.urdf (robot description, URDF)
Before this commit: robot default_cube, 1 links, 0 joints
Links:
- removed link cube_link
- added link generic_cube_link, mass 1.0; collision mesh filename=package://Generic_Cube/meshes/recube.stl scale=0.01 0.01 0.01; visual mesh filename=package://Generic_Cube/meshes/recube.stl scale=0.01 0.01 0.01

Commit message: resize recube

File: Generic_Objects/Generic_Cube/urdf/recube.urdf (robot description, URDF)
Before this commit: robot generic_cube, 1 links, 0 joints
Links:
- link generic_cube_link: geometry collision mesh filename=package://Generic_Cube/meshes/recube.stl scale=0.001 0.001 0.001; visual mesh filename=package://Generic_Cube/meshes/recube.stl scale=0.001 0.001 0.001
