Commit message: change name again to cube

File: Generic_Objects/Generic_Cube/urdf/recubedd.urdf (robot description, URDF)
Before this commit: robot generic_cube, 1 links, 0 joints
Links:
- link generic_cube_link: geometry collision mesh filename=package://Generic_Cube/meshes/recube.stl scale=0.01 0.01 0.01; visual mesh filename=package://Generic_Cube/meshes/recube.stl scale=0.01 0.01 0.01
