Commit message: another cube

File: Generic_Objects/Generic_Cube/urdf/cube1m.urdf (robot description, URDF)
Before this commit: robot generic_cube, 1 links, 0 joints
Links:
- removed link generic_cube_link
- added link cube_link, mass 1.0; collision mesh filename=package://Generic_Cube/meshes/cube1m.stl scale=0.01 0.01 0.01; visual mesh filename=package://Generic_Cube/meshes/cube1m.stl scale=0.01 0.01 0.01
