Commit message: cube again 2

File: Generic_Objects/Generic_Cube/urdf/cube1hm.urdf (robot description, URDF)
Before this commit: robot generic_cube, 1 links, 0 joints
Links:
- link cube_link: geometry collision mesh filename=package://Generic_Cube/meshes/cube1hm.stl scale=0.01 0.01 0.01; visual mesh filename=package://Generic_Cube/meshes/cube1hm.stl scale=0.01 0.01 0.01
