Commit message: generic table flipped faces

File: Generic_Objects/Generic_Table/urdf/generictable2.urdf (robot description, URDF)
Before this commit: robot generic_table, 1 links, 0 joints
Links:
- link table_link: geometry collision mesh filename=package://Generic_Table/meshes/generictable2.stl scale=1.0 1.0 1.0; visual mesh filename=package://Generic_Table/meshes/generictable2.stl scale=1.0 1.0 1.0
