Commit message: Box2 flaps out

File: Generic_Objects/Generic_Box_flaps_out/urdf/Generic_Box.urdf (robot description, URDF)
Before this commit: robot open_box_flaps_out, 1 links, 0 joints
Links:
- link box_link: mass 0.5 -> 2.0; geometry collision mesh filename=package://Generic_Box_flaps_out/meshes/Generic Box.stl scale=1.0 1.0 1.0; visual mesh filename=package://Generic_Box_flaps_out/meshes/Generic Box.stl scale=1.0 1.0 1.0
