Commit message: changing value urdf

File: Universal_Robots/UR5_Robot/urdf/ur5robot.urdf (robot description, URDF)
Before this commit: robot universal-robot-ur5, 9 links, 8 joints
Joints:
- joint elbow_joint: limit lower=-6.2831853 upper=6.2831853 effort=150.0 velocity=3.14159265 -> lower=-3.14159265 upper=3.14159265 effort=150.0 velocity=3.14159265
- joint shoulder_lift_joint: limit lower=-6.2831853 upper=6.2831853 effort=150.0 velocity=3.14159265 -> lower=-3.14159265 upper=3.14159265 effort=150.0 velocity=3.14159265
- joint shoulder_pan_joint: limit lower=-6.2831853 upper=6.2831853 effort=150.0 velocity=3.14159265 -> lower=-3.14159265 upper=3.14159265 effort=150.0 velocity=3.14159265
