Commit message: UR_changeneup

File: Universal_Robots/UR5/ur5robot.urdf (robot description, URDF)
Before this commit: robot universal-robot-ur5, 9 links, 8 joints
Links:
- link base_link: geometry collision mesh filename=package://meshes/ur5/collision/Base.dae; visual mesh filename=package://meshes/ur5/visual/Base.dae
- link forearm_link: geometry collision mesh filename=package://meshes/ur5/collision/Forearm.dae; visual mesh filename=package://meshes/ur5/visual/Forearm.dae
- link shoulder_link: geometry collision mesh filename=package://meshes/ur5/collision/Shoulder.dae; visual mesh filename=package://meshes/ur5/visual/Shoulder.dae
- link upper_arm_link: geometry collision mesh filename=package://meshes/ur5/collision/UpperArm.dae; visual mesh filename=package://meshes/ur5/visual/UpperArm.dae
- link wrist_1_link: geometry collision mesh filename=package://meshes/ur5/collision/Wrist1.dae; visual mesh filename=package://meshes/ur5/visual/Wrist1.dae
- link wrist_2_link: geometry collision mesh filename=package://meshes/ur5/collision/Wrist2.dae; visual mesh filename=package://meshes/ur5/visual/Wrist2.dae
- link wrist_3_link: geometry collision mesh filename=package://meshes/ur5/collision/Wrist3.dae; visual mesh filename=package://meshes/ur5/visual/Wrist3.dae

Commit message: retry UR5

File: Universal_Robots/UR5/ur5robot.urdf (robot description, URDF)
Before this commit: robot universal-robot-ur5, 9 links, 8 joints
Links:
- link base_link: geometry collision mesh filename=package://UR5/meshes/ur5/collision/Base.dae; visual mesh filename=package://UR5/meshes/ur5/visual/Base.dae
- link forearm_link: geometry collision mesh filename=package://UR5/meshes/ur5/collision/Forearm.dae; visual mesh filename=package://UR5/meshes/ur5/visual/Forearm.dae
- link shoulder_link: geometry collision mesh filename=package://UR5/meshes/ur5/collision/Shoulder.dae; visual mesh filename=package://UR5/meshes/ur5/visual/Shoulder.dae
- link upper_arm_link: geometry collision mesh filename=package://UR5/meshes/ur5/collision/UpperArm.dae; visual mesh filename=package://UR5/meshes/ur5/visual/UpperArm.dae
- link wrist_1_link: geometry collision mesh filename=package://UR5/meshes/ur5/collision/Wrist1.dae; visual mesh filename=package://UR5/meshes/ur5/visual/Wrist1.dae
- link wrist_2_link: geometry collision mesh filename=package://UR5/meshes/ur5/collision/Wrist2.dae; visual mesh filename=package://UR5/meshes/ur5/visual/Wrist2.dae
- link wrist_3_link: geometry collision mesh filename=package://UR5/meshes/ur5/collision/Wrist3.dae; visual mesh filename=package://UR5/meshes/ur5/visual/Wrist3.dae
