Commit message: BRCD3

File: Duatic_R/Bot_Baracuda12/Brcd12.urdf (robot description, URDF)
Before this commit: robot dynaarm, 11 links, 10 joints
Links:
- link base: geometry collision mesh filename=package://Bot_Baracuda12/meshes/collision/base_mesh.stl scale=1.0 1.0 1.0; visual mesh filename=package://Bot_Baracuda12/meshes/visual/base_mesh.dae scale=1.0 1.0 1.0
- link elbow: geometry collision mesh filename=package://Bot_Baracuda12/meshes/collision/elbow_mesh.stl scale=1.0 1.0 1.0; visual mesh filename=package://Bot_Baracuda12/meshes/visual/elbow_mesh.dae scale=1.0 1.0 1.0
- link forearm: geometry collision mesh filename=package://Bot_Baracuda12/meshes/collision/forearm_mesh.stl scale=1.0 1.0 1.0; visual mesh filename=package://Bot_Baracuda12/meshes/visual/forearm_mesh.dae scale=1.0 1.0 1.0
- link shoulder: geometry collision mesh filename=package://Bot_Baracuda12/meshes/collision/shoulder_mesh.stl scale=1.0 1.0 1.0; visual mesh filename=package://Bot_Baracuda12/meshes/visual/shoulder_mesh.dae scale=1.0 1.0 1.0
- link upperarm: geometry collision mesh filename=package://Bot_Baracuda12/meshes/collision/upperarm_mesh.stl scale=1.0 1.0 1.0; visual mesh filename=package://Bot_Baracuda12/meshes/visual/upperarm_mesh.dae scale=1.0 1.0 1.0
- link wrist_1: geometry collision mesh filename=package://Bot_Baracuda12/meshes/collision/wrist1_mesh.stl scale=1.0 1.0 1.0; visual mesh filename=package://Bot_Baracuda12/meshes/visual/wrist1_mesh.dae scale=1.0 1.0 1.0
- link wrist_2: geometry collision mesh filename=package://Bot_Baracuda12/meshes/collision/wrist2_mesh.stl scale=1.0 1.0 1.0; visual mesh filename=package://Bot_Baracuda12/meshes/visual/wrist2_mesh.dae scale=1.0 1.0 1.0
