Commit message: DELETE1

File: Holybro/PX4Vision/urdf/frankenpx4.urdf (robot description, URDF)
Before this commit: robot px4_vision, 1 links, 0 joints
Links:
- link base_link: geometry collision mesh filename=package://PX4Vision/meshes/px4Lidl.stl scale=0.001 0.001 0.001; visual mesh filename=package://PX4Vision/meshes/px4Lidl.stl scale=0.001 0.001 0.001
