Commit message: NewSO101toDEL

File: FFD/urdf/NEWtoDELETEso101_old_calib.urdf (robot description, URDF)
Before this commit: robot so101_old_calib, 7 links, 6 joints
Links:
- link base: geometry collision mesh filename=package://FFD/assets/base_motor_holder_so101_v1.stl; collision mesh filename=package://FFD/assets/base_so101_v2.stl
- link gripper: geometry collision mesh filename=package://FFD/assets/sts3215_03a_v1.stl; collision mesh filename=package://FFD/assets/wrist_roll_follower_so101_v1.stl
- link jaw: geometry collision mesh filename=package://FFD/assets/moving_jaw_so101_v1.stl; visual mesh filename=package://FFD/assets/moving_jaw_so101_v1.stl
- link lower_arm: geometry collision mesh filename=package://FFD/assets/motor_holder_so101_wrist_v1.stl; collision mesh filename=package://FFD/assets/sts3215_03a_v1.stl
- link shoulder: geometry collision mesh filename=package://FFD/assets/motor_holder_so101_base_v1.stl; collision mesh filename=package://FFD/assets/rotation_pitch_so101_v1.stl
- link upper_arm: geometry collision mesh filename=package://FFD/assets/sts3215_03a_v1.stl; collision mesh filename=package://FFD/assets/upper_arm_so101_v1.stl
- link wrist: geometry collision mesh filename=package://FFD/assets/sts3215_03a_no_horn_v1.stl; collision mesh filename=package://FFD/assets/wrist_roll_pitch_so101_v2.stl
