Commit message: To_F_DEMO

File: Agilox_AgiloxOFL/urdf/ofl_robot.urdf (robot description, URDF)
Before this commit: robot ofl_robot, 2 links, 1 joints
Links:
- link base_link: geometry collision mesh filename=package://Agilox_AgiloxOFL/meshes/body1.stl scale=1.0 1.0 1.0; visual mesh filename=package://Agilox_AgiloxOFL/meshes/body1.stl scale=1.0 1.0 1.0
- link skates_link: geometry collision mesh filename=package://Agilox_AgiloxOFL/meshes/skates1.stl scale=1.0 1.0 1.0; visual mesh filename=package://Agilox_AgiloxOFL/meshes/skates1.stl scale=1.0 1.0 1.0

Commit message: UpdateMeshes

File: Agilox_AgiloxOFL/urdf/ofl_robot.urdf (robot description, URDF)
Before this commit: robot ofl_robot, 2 links, 1 joints
Links:
- link base_link: geometry collision mesh filename=package://Agilox_AgiloxOFL/meshes/body2.stl scale=1.0 1.0 1.0; visual mesh filename=package://Agilox_AgiloxOFL/meshes/body2.stl scale=1.0 1.0 1.0
