Commit message: update

File: Amrobotics_Otto1500/OTTO/urdf/otto1500.urdf (robot description, URDF)
Before this commit: robot otto1500, 1 links, 0 joints
Links:
- link base_link: geometry collision mesh filename=package://Amrobotics_Otto1500/OTTO/meshes/otto1500.stl scale=1.0 1.0 1.0; visual mesh filename=package://Amrobotics_Otto1500/OTTO/meshes/otto1500.stl scale=1.0 1.0 1.0
