Commit message: DelUp

File: mir_250/urdf/mir.urdf (robot description, URDF)
Before this commit: robot mir, 19 links, 18 joints
Links:
- link back_laser_link: geometry collision mesh filename=package://mir_250/meshes/visual/sick_lms-100.stl; visual mesh filename=package://mir_250/meshes/visual/sick_lms-100.stl
- link base_link: geometry collision mesh filename=package://mir_250/meshes/collision/mir_250_base.stl; visual mesh filename=package://mir_250/meshes/visual/mir_250_base.stl
- link bl_caster_rotation_link: geometry collision mesh filename=package://mir_250/meshes/collision/caster_wheel_base.stl; visual mesh filename=package://mir_250/meshes/visual/caster_wheel_base.stl
- link br_caster_rotation_link: geometry collision mesh filename=package://mir_250/meshes/collision/caster_wheel_base.stl; visual mesh filename=package://mir_250/meshes/visual/caster_wheel_base.stl
- link fl_caster_rotation_link: geometry collision mesh filename=package://mir_250/meshes/collision/caster_wheel_base.stl; visual mesh filename=package://mir_250/meshes/visual/caster_wheel_base.stl
- link fr_caster_rotation_link: geometry collision mesh filename=package://mir_250/meshes/collision/caster_wheel_base.stl; visual mesh filename=package://mir_250/meshes/visual/caster_wheel_base.stl
- link front_laser_link: geometry collision mesh filename=package://mir_250/meshes/visual/sick_lms-100.stl; visual mesh filename=package://mir_250/meshes/visual/sick_lms-100.stl
