Commit message: Newxml

File: Agile_X_Robotics/tracer_20/urdf/tracer_v1.urdf (robot description, URDF)
Before this commit: robot tracer_v1, 12 links, 11 joints
Links:
- link base_link: geometry collision mesh filename=package://Agile_X_Robotics/tracer_20/meshes/tracer_base_lin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; visual mesh filename=package://Agile_X_Robotics/tracer_20/meshes/tracer_base_lin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
- link fl_castor_link: geometry visual mesh filename=package://Agile_X_Robotics/tracer_20/meshes/castor_joint.stl
- link fl_wheel_link: geometry collision mesh filename=package://Agile_X_Robotics/tracer_20/meshes/castor.stl; visual mesh filename=package://Agile_X_Robotics/tracer_20/meshes/castor.stl
- link fr_castor_link: geometry visual mesh filename=package://Agile_X_Robotics/tracer_20/meshes/castor_joint.stl
- link fr_wheel_link: geometry collision mesh filename=package://Agile_X_Robotics/tracer_20/meshes/castor.stl; visual mesh filename=package://Agile_X_Robotics/tracer_20/meshes/castor.stl
- link left_wheel_link: geometry collision mesh filename=package://Agile_X_Robotics/tracer_20/meshes/tracer_wheel.stl; visual mesh filename=package://Agile_X_Robotics/tracer_20/meshes/tracer_wheel.stl
- link right_wheel_link: geometry collision mesh filename=package://Agile_X_Robotics/tracer_20/meshes/tracer_wheel.stl; visual mesh filename=package://Agile_X_Robotics/tracer_20/meshes/tracer_wheel.stl
- link rl_castor_link: geometry visual mesh filename=package://Agile_X_Robotics/tracer_20/meshes/castor_joint.stl
- link rl_wheel_link: geometry collision mesh filename=package://Agile_X_Robotics/tracer_20/meshes/castor.stl; visual mesh filename=package://Agile_X_Robotics/tracer_20/meshes/castor.stl
- link rr_castor_link: geometry visual mesh filename=package://Agile_X_Robotics/tracer_20/meshes/castor_joint.stl
- link rr_wheel_link: geometry collision mesh filename=package://Agile_X_Robotics/tracer_20/meshes/castor.stl; visual mesh filename=package://Agile_X_Robotics/tracer_20/meshes/castor.stl

Commit message: Urdf2

File: Agile_X_Robotics/tracer_20/urdf/tracer_v1.urdf (robot description, URDF)
Before this commit: robot tracer_v1, 12 links, 11 joints
Links:
- link base_link: geometry collision mesh filename=../meshes/tracer_base_link.stl; visual mesh filename=../meshes/tracer_base_link.stl
- link fl_castor_link: geometry visual mesh filename=../meshes/castor_joint.stl
- link fl_wheel_link: geometry collision mesh filename=../meshes/castor.stl; visual mesh filename=../meshes/castor.stl
- link fr_castor_link: geometry visual mesh filename=../meshes/castor_joint.stl
- link fr_wheel_link: geometry collision mesh filename=../meshes/castor.stl; visual mesh filename=../meshes/castor.stl
- link left_wheel_link: geometry collision mesh filename=../meshes/tracer_wheel.stl; visual mesh filename=../meshes/tracer_wheel.stl
- link right_wheel_link: geometry collision mesh filename=../meshes/tracer_wheel.stl; visual mesh filename=../meshes/tracer_wheel.stl
- link rl_castor_link: geometry visual mesh filename=../meshes/castor_joint.stl
- link rl_wheel_link: geometry collision mesh filename=../meshes/castor.stl; visual mesh filename=../meshes/castor.stl
- link rr_castor_link: geometry visual mesh filename=../meshes/castor_joint.stl
- link rr_wheel_link: geometry collision mesh filename=../meshes/castor.stl; visual mesh filename=../meshes/castor.stl
