Commit message: Kukared

File: KUKA/KR70/urdf/kr70_r2100.urdf (robot description, URDF)
Before this commit: robot kr70_r2100, 11 links, 10 joints
Links:
- link base_link: geometry collision mesh filename=package://KUKA/KR70/meshes/collision/base_link.stl; visual mesh filename=package://KUKA/KR70/meshes/visual/base_link.stl
- link link_1: geometry collision mesh filename=package://KUKA/KR70/meshes/collision/link_1.stl; visual mesh filename=package://KUKA/KR70/meshes/visual/link_1.stl
- link link_2: geometry collision mesh filename=package://KUKA/KR70/meshes/collision/link_2.stl; visual mesh filename=package://KUKA/KR70/meshes/visual/link_2.stl
- link link_3: geometry collision mesh filename=package://KUKA/KR70/meshes/collision/link_3.stl; visual mesh filename=package://KUKA/KR70/meshes/visual/link_3.stl
- link link_4: geometry collision mesh filename=package://KUKA/KR70/meshes/collision/link_4.stl; visual mesh filename=package://KUKA/KR70/meshes/visual/link_4.stl
- link link_5: geometry collision mesh filename=package://KUKA/KR70/meshes/collision/link_5.stl; visual mesh filename=package://KUKA/KR70/meshes/visual/link_5.stl
- link link_6: geometry collision mesh filename=package://KUKA/KR70/meshes/collision/link_6.stl; visual mesh filename=package://KUKA/KR70/meshes/visual/link_6.stl

Commit message: pnrmNew

File: KUKA/KR70/urdf/kr70_r2100.urdf (robot description, URDF)
Before this commit: robot kr70_r2100, 11 links, 10 joints
Links:
- link base_link: geometry collision mesh filename=package://KUKA_LBR/KR70/meshes/collision/base_link.stl; visual mesh filename=package://KUKA_LBR/KR70/meshes/visual/base_link.stl
- link link_1: geometry collision mesh filename=package://KUKA_LBR/KR70/meshes/collision/link_1.stl; visual mesh filename=package://KUKA_LBR/KR70/meshes/visual/link_1.stl
- link link_2: geometry collision mesh filename=package://KUKA_LBR/KR70/meshes/collision/link_2.stl; visual mesh filename=package://KUKA_LBR/KR70/meshes/visual/link_2.stl
- link link_3: geometry collision mesh filename=package://KUKA_LBR/KR70/meshes/collision/link_3.stl; visual mesh filename=package://KUKA_LBR/KR70/meshes/visual/link_3.stl
- link link_4: geometry collision mesh filename=package://KUKA_LBR/KR70/meshes/collision/link_4.stl; visual mesh filename=package://KUKA_LBR/KR70/meshes/visual/link_4.stl
- link link_5: geometry collision mesh filename=package://KUKA_LBR/KR70/meshes/collision/link_5.stl; visual mesh filename=package://KUKA_LBR/KR70/meshes/visual/link_5.stl
- link link_6: geometry collision mesh filename=package://KUKA_LBR/KR70/meshes/collision/link_6.stl; visual mesh filename=package://KUKA_LBR/KR70/meshes/visual/link_6.stl

File: openarm/urdf/NewOAr_bimanual.urdf (robot description, URDF)
Before this commit: robot openarm, 24 links, 23 joints
Joints:
- removed joint openarm_left_finger1_joint
- removed joint openarm_left_finger2_joint
- removed joint openarm_right_finger1_joint
- removed joint openarm_right_finger2_joint
- added joint openarm_left_finger_joint1: type prismatic, parent openarm_left_hand, child openarm_left_finger1, origin xyz=0.0 0.0 0.075 rpy=0 0 0, axis 0 1 0, limit lower=0.0 upper=0.044 effort=333 velocity=10.0
- added joint openarm_left_finger_joint2: type prismatic, parent openarm_left_hand, child openarm_left_finger2, origin xyz=0.0 0.0 0.075 rpy=0 0 0, axis 0 -1 0, limit lower=0.0 upper=0.044 effort=333 velocity=10.0
- added joint openarm_right_finger_joint1: type prismatic, parent openarm_right_hand, child openarm_right_finger1, origin xyz=0.0 0.0 0.075 rpy=0 0 0, axis 0 1 0, limit lower=0.0 upper=0.044 effort=333 velocity=10.0
- added joint openarm_right_finger_joint2: type prismatic, parent openarm_right_hand, child openarm_right_finger2, origin xyz=0.0 0.0 0.075 rpy=0 0 0, axis 0 -1 0, limit lower=0.0 upper=0.044 effort=333 velocity=10.0
