Commit message: newURDFSO1

File: Lerobot/SO101/urdf/CybModSO101.urdf (robot description, URDF)
Before this commit: robot so101_new_calib, 7 links, 6 joints
Links:
- link base: geometry collision mesh filename=package://Lerobot/SO101/assets/base_motor_holder_so101_v1.s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; collision mesh filename=package://Lerobot/SO101/assets/base_so101_v2.stl
- link gripper: geometry collision mesh filename=package://Lerobot/SO101/assets/sts3215_03a_v1.stl; collision mesh filename=package://Lerobot/SO101/assets/wrist_roll_follower_so101_v1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
- link jaw: geometry collision mesh filename=package://Lerobot/SO101/assets/moving_jaw_so101_v1.stl; visual mesh filename=package://Lerobot/SO101/assets/moving_jaw_so101_v1.stl
- link lower_arm: geometry collision mesh filename=package://Lerobot/SO101/assets/motor_holder_so101_wrist_v1.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; collision mesh filename=package://Lerobot/SO101/assets/sts3215_03a_v1.stl
- link shoulder: geometry collision mesh filename=package://Lerobot/SO101/assets/motor_holder_so101_base_v1.s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; collision mesh filename=package://Lerobot/SO101/assets/rotation_pitch_so101_v1.stl
- link upper_arm: geometry collision mesh filename=package://Lerobot/SO101/assets/sts3215_03a_v1.stl; collision mesh filename=package://Lerobot/SO101/assets/upper_arm_so101_v1.stl
- link wrist: geometry collision mesh filename=package://Lerobot/SO101/assets/sts3215_03a_no_horn_v1.stl; collision mesh filename=package://Lerobot/SO101/assets/wrist_roll_pitch_so101_v2.stl
