Commit message: Change mesh file format from STL to OBJ

File: Environments/SAP_warehouse/urdf/sap_warehouse.urdf (robot description, URDF)
Before this commit: robot sap_warehouse, 2 links, 1 joints
Links:
- link sap_warehouse_link: geometry collision mesh filename=package://Environments/SAP_warehouse/meshes/sap_warehouse.s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; visual mesh filename=package://Environments/SAP_warehouse/meshes/sap_warehouse.o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
