Commit message: UpdateCYp

File: Generic_Objects/Cyber_Pad/urdf/CyPad.urdf (robot description, URDF)
Before this commit: robot CyPad, 1 links, 0 joints
Links:
- link base_link: geometry collision mesh filename=package://Cyber_Pad/meshes/collision/CyPad2.stl; visual mesh filename=package://Cyber_Pad/meshes/visual/CyPad2.obj
