Commit message: Gemini355Lg

File: Orbbec/gemini_335lg/urdf/gemini_335lg.urdf (robot description, URDF)
Before this commit: robot gemini_335lg, 6 links, 5 joints
Links:
- link camera_link: geometry collision box size=0.124 0.029 0.038; visual mesh filename=package://gemini_335lg/meshes/Gemini355Lg.stl scale=0.001 0.001 0.001
