Commit message: add floor and wall meshes

File: Generic_Objects/Floor/urdf/floor.urdf (robot description, URDF)
Before this commit: robot wall, 2 links, 1 joints
Links:
- link base_link: geometry collision mesh filename=../meshes/floor.stl; visual mesh filename=../meshes/floor.obj

Commit message: fix floor

File: Generic_Objects/Floor/urdf/floor.urdf (robot description, URDF)
Before this commit: robot floor, 2 links, 1 joints
Links:
- link base_link: geometry collision mesh filename=../meshes/floor.obj; visual mesh filename=../meshes/floor.obj
