Commit message: fix DJI mavic URDF

File: DJI_bot/DJI-Mavic-3-Enterprise/urdf/dji_drone.urdf (robot description, URDF)
Before this commit: robot sentinel_drone, 11 links, 10 joints
Links:
- link base_link: geometry collision box size=0.35 0.28 0.11; visual mesh filename=../meshes/body.stl scale=0.015 0.015 0.015
- link prop_fl: geometry visual mesh filename=../meshes/prop_fl.stl scale=0.015 0.015 0.015
- link prop_fr: geometry visual mesh filename=../meshes/prop_fr.stl scale=0.015 0.015 0.015
- link prop_rl: geometry visual mesh filename=../meshes/prop_rl.stl scale=0.015 0.015 0.015
- link prop_rr: geometry visual mesh filename=../meshes/prop_rr.stl scale=0.015 0.015 0.015
