Commit message: actuate ugv

File: DJI_bot/Mavic-3-Enterprise/urdf/dji_drone.urdf (robot description, URDF)
Before this commit: robot sentinel_drone, 11 links, 10 joints
Links:
- link base_link: geometry collision box size=0.28 0.35 0.11; visual mesh filename=../meshes/body.stl scale=0.015 0.015 0.015
Joints:
- joint arm_fl_joint: origin xyz=-0.1207 0.0737 0.008 -> xyz=0.0737 0.1207 0.008
- joint arm_fr_joint: origin xyz=0.1207 0.0737 0.0081 -> xyz=0.0737 -0.1207 0.0081
- joint arm_rl_joint: origin xyz=-0.0956 -0.1081 0.0029 -> xyz=-0.1081 0.0956 0.0029
- joint arm_rr_joint: origin xyz=0.0956 -0.1081 0.0029 -> xyz=-0.1081 -0.0956 0.0029
- joint camera_joint: origin xyz=0 0.1585 0.0091 rpy=0 0 0 -> xyz=0.1585 0 0.0091 rpy=0 0 0
- joint payload_joint: origin xyz=0 0.1585 -0.0209 rpy=0 0 0 -> xyz=0.1585 0 -0.0209 rpy=0 0 0
- joint prop_fl_joint: origin xyz=-0.2414 0.1474 0.016 -> xyz=0.1474 0.2414 0.016
- joint prop_fr_joint: origin xyz=0.2414 0.1474 0.0162 -> xyz=0.1474 -0.2414 0.0162
- joint prop_rl_joint: origin xyz=-0.1912 -0.2162 0.0057 -> xyz=-0.2162 0.1912 0.0057
- joint prop_rr_joint: origin xyz=0.1912 -0.2162 0.0058 -> xyz=-0.2162 -0.1912 0.0058

File: Waveshare__/UGVBeast__/urdf/NEWDATAUGV_BeastUGV_.urdf (robot description, URDF)
Before this commit: robot ugv_beast_pt, 10 links, 9 joints
Links:
- link base_link: geometry collision mesh filename=package://UGVBeast__/meshes/ugv_body.stl scale=0.001 0.001 0.001; visual mesh filename=package://UGVBeast__/meshes/ugv_body.stl scale=0.001 0.001 0.001
- link pt_link1: geometry collision mesh filename=package://UGVBeast__/meshes/pt_link1.stl scale=0.001 0.001 0.001; visual mesh filename=package://UGVBeast__/meshes/pt_link1.stl scale=0.001 0.001 0.001
- link pt_link2: geometry collision mesh filename=package://UGVBeast__/meshes/pt_link2.stl scale=0.001 0.001 0.001; visual mesh filename=package://UGVBeast__/meshes/pt_link2.stl scale=0.001 0.001 0.001
Joints:
- joint camera_joint: origin xyz=0.02 0 0 rpy=0 0 0 -> xyz=0.03 0 0.01 rpy=0 0 0
- joint lidar_joint: origin xyz=0 0 0.2 rpy=0 0 0 -> xyz=0 0 0.14 rpy=0 0 0
- joint pt_base_link_to_pt_link1: origin xyz=0.1 0 0.15 rpy=0 0 0 -> xyz=-0.0035 0 0.136 rpy=0 0 0
- joint pt_link1_to_pt_link2: origin xyz=0 0 0.05 rpy=0 0 0 -> xyz=-0.0005 0 0.052 rpy=0 0 0
