Commit message: fix urdf

File: Waveshare__/UGVBeast__/urdf/NEWDATAUGV_BeastUGV_.urdf (robot description, URDF)
Before this commit: robot ugv_beast_pt, 10 links, 9 joints
Links:
- link base_link: geometry collision mesh filename=../meshes/ugv_body.stl scale=0.001 0.001 0.001; visual mesh filename=../meshes/ugv_body.stl scale=0.001 0.001 0.001
- link pt_link1: geometry collision mesh filename=../meshes/pt_link1.stl scale=0.001 0.001 0.001; visual mesh filename=../meshes/pt_link1.stl scale=0.001 0.001 0.001
- link pt_link2: geometry collision mesh filename=../meshes/pt_link2.stl scale=0.001 0.001 0.001; visual mesh filename=../meshes/pt_link2.stl scale=0.001 0.001 0.001
