Commit message: dji pro with propellers

File: DJI_bot/4DJIMINI4PRO/urdf/DJI4p.urdf (robot description, URDF)
Before this commit: robot dji_mini_4_pro, 1 links, 0 joints
Links:
- added link prop_back_left, mass 0.001; collision mesh filename=package://4DJIMINI4PRO/meshes/prop_back_left.stl scale=0.01 0.01 0.01; visual mesh filename=package://4DJIMINI4PRO/meshes/prop_back_left.stl scale=0.01 0.01 0.01
- added link prop_back_right, mass 0.001; collision mesh filename=package://4DJIMINI4PRO/meshes/prop_back_right.stl scale=0.01 0.01 0.01; visual mesh filename=package://4DJIMINI4PRO/meshes/prop_back_right.stl scale=0.01 0.01 0.01
- added link prop_front_left, mass 0.001; collision mesh filename=package://4DJIMINI4PRO/meshes/prop_front_left.stl scale=0.01 0.01 0.01; visual mesh filename=package://4DJIMINI4PRO/meshes/prop_front_left.stl scale=0.01 0.01 0.01
- added link prop_front_right, mass 0.001; collision mesh filename=package://4DJIMINI4PRO/meshes/prop_front_right.stl scale=0.01 0.01 0.01; visual mesh filename=package://4DJIMINI4PRO/meshes/prop_front_right.stl scale=0.01 0.01 0.01
- link base_link: mass 0.249 -> 0.245; geometry collision mesh filename=package://4DJIMINI4PRO/meshes/body.stl scale=0.01 0.01 0.01; visual mesh filename=package://4DJIMINI4PRO/meshes/body.stl scale=0.01 0.01 0.01
Joints:
- added joint prop_back_left_joint: type continuous, parent base_link, child prop_back_left, origin xyz=-0.07680 -0.08956 0.02630 rpy=0 0 0, axis -0.16047 0.30221 0.93964
- added joint prop_back_right_joint: type continuous, parent base_link, child prop_back_right, origin xyz=0.07665 -0.08981 0.02489 rpy=0 0 0, axis 0.22021 0.21100 0.95236
- added joint prop_front_left_joint: type continuous, parent base_link, child prop_front_left, origin xyz=-0.10764 0.06722 -0.00450 rpy=0 0 0, axis -0.10884 0.23674 0.96546
- added joint prop_front_right_joint: type continuous, parent base_link, child prop_front_right, origin xyz=0.11354 0.05739 -0.00263 rpy=0 0 0, axis 0.03749 0.18959 0.98115
