Commit message: dji mini 3 pro with propellers

File: DJI_bot/DJIMini3Pro/urdf/DJImini3.urdf (robot description, URDF)
Before this commit: robot dji_mini_3_pro, 1 links, 0 joints
Links:
- added link prop_back_left, mass 0.001; collision mesh filename=../meshes/prop_back_left.stl scale=1.0 1.0 1.0; visual mesh filename=../meshes/prop_back_left.stl scale=1.0 1.0 1.0
- added link prop_back_right, mass 0.001; collision mesh filename=../meshes/prop_back_right.stl scale=1.0 1.0 1.0; visual mesh filename=../meshes/prop_back_right.stl scale=1.0 1.0 1.0
- added link prop_front_left, mass 0.001; collision mesh filename=../meshes/prop_front_left.stl scale=1.0 1.0 1.0; visual mesh filename=../meshes/prop_front_left.stl scale=1.0 1.0 1.0
- added link prop_front_right, mass 0.001; collision mesh filename=../meshes/prop_front_right.stl scale=1.0 1.0 1.0; visual mesh filename=../meshes/prop_front_right.stl scale=1.0 1.0 1.0
- link base_link: mass 0.249 -> 0.245; geometry collision mesh filename=../meshes/body.stl scale=1.0 1.0 1.0; visual mesh filename=../meshes/body.stl scale=1.0 1.0 1.0
Joints:
- added joint prop_back_left_joint: type continuous, parent base_link, child prop_back_left, origin xyz=-0.082 0.115 0.046 rpy=0 0 0, axis -0.31966 -0.11255 0.94082
- added joint prop_back_right_joint: type continuous, parent base_link, child prop_back_right, origin xyz=0.081 0.115 0.046 rpy=0 0 0, axis 0.10676 -0.25905 0.95995
- added joint prop_front_left_joint: type continuous, parent base_link, child prop_front_left, origin xyz=-0.114 -0.036 0.020 rpy=0 0 0, axis 0.11694 -0.16841 0.97876
- added joint prop_front_right_joint: type continuous, parent base_link, child prop_front_right, origin xyz=0.113 -0.036 0.020 rpy=0 0 0, axis -0.11730 -0.16817 0.97875

Commit message: Update DJI Mini 3 Pro separated meshes

File: DJI_bot/DJIMini3Pro/urdf/DJImini3.urdf (robot description, URDF)
Before this commit: robot dji_mini_3_pro, 5 links, 4 joints
Links:
- added link camera_gimbal, mass 0.010; collision mesh filename=../meshes/camera_gimbal.stl scale=1.0 1.0 1.0; visual mesh filename=../meshes/camera_gimbal.stl scale=1.0 1.0 1.0
- link base_link: mass 0.245 -> 0.235
Joints:
- added joint camera_gimbal_pitch_joint: type continuous, parent base_link, child camera_gimbal, origin xyz=-0.001653 -0.033692 0.013606 rpy=0 0 0, axis 1 0 0
