Commit message: h_urdf_upload3

File: Hitachi/hitachi_model/urdf/hitachi.urdf (robot description, URDF)
Before this commit: robot hitachi_model, 1 links, 0 joints
Links:
- link base_link: geometry collision mesh filename=package://hitachi_model/meshes/Capture.dae scale=0.1 0.1 0.1; visual mesh filename=package://hitachi_model/meshes/Capture.dae scale=0.1 0.1 0.1

Commit message: h_urdf_upload4

File: Hitachi/hitachi_model/urdf/hitachi.urdf (robot description, URDF)
Before this commit: robot hitachi_model, 1 links, 0 joints
Links:
- link base_link: geometry collision mesh filename=package://hitachi_model/meshes/Capture.dae scale=0.5 0.5 0.5; visual mesh filename=package://hitachi_model/meshes/Capture.dae scale=0.5 0.5 0.5
