Commit message: add collision for the substation

File: Environments/Substation/urdf/substation.urdf (robot description, URDF)
Before this commit: robot substation, 1 links, 0 joints
Links:
- link substation_base_link: geometry collision mesh filename=package://Substation/meshes/substation_collision.stl scale=1.0 1.0 1.0; visual mesh filename=package://Substation/meshes/substation.stl scale=1.0 1.0 1.0
