Commit message: fix stls

File: Modalai/Starling_Max/urdf/starling_max.urdf (robot description, URDF)
Before this commit: robot starling_max, 5 links, 4 joints
Joints:
- joint prop_fl_joint: origin xyz=0.2758 0.2666 0.0684 -> xyz=0.5999 0.4552 0.1702
- joint prop_fr_joint: origin xyz=0.3318 -0.3208 0.0524 -> xyz=0.6012 -0.4609 0.1598
- joint prop_rl_joint: origin xyz=-0.3369 0.3215 0.0511 -> xyz=-0.6051 0.4528 0.1237
- joint prop_rr_joint: origin xyz=-0.3367 -0.3221 0.0521 -> xyz=-0.592 -0.4553 0.093

Commit message: update size

File: Modalai/Starling_Max/urdf/starling_max.urdf (robot description, URDF)
Before this commit: robot starling_max, 5 links, 4 joints
Links:
- link base_link: geometry collision box size=0.1215 0.0942 0.0546; visual mesh filename=../meshes/body.stl scale=1.0 1.0 1.0
Joints:
- joint prop_fl_joint: origin xyz=0.5999 0.4552 0.1702 -> xyz=0.0565 0.0429 0.016
- joint prop_fr_joint: origin xyz=0.6012 -0.4609 0.1598 -> xyz=0.0566 -0.0434 0.0151
- joint prop_rl_joint: origin xyz=-0.6051 0.4528 0.1237 -> xyz=-0.057 0.0426 0.0117
- joint prop_rr_joint: origin xyz=-0.592 -0.4553 0.093 -> xyz=-0.0558 -0.0429 0.0088
