Commit message: better amcrest

File: Amcrest/IP4M-1041/urdf/IP4M-1041.urdf (robot description, URDF)
Before this commit: robot amcrest_ip4m_1041, 4 links, 3 joints
Links:
- removed link amcrest_camera_link
- added link amcrest_camera_frame
- added link amcrest_tilt_link, mass 0.070; collision mesh filename=../meshes/IP4M_1041_tilt_collision.stl; visual mesh filename=../meshes/IP4M_1041_tilt_visual.obj
- link amcrest_base_link: mass 0.140 -> 0.120; geometry collision mesh filename=../meshes/IP4M_1041_base_collision.stl; visual mesh filename=../meshes/IP4M_1041_base_visual.obj
- link amcrest_pan_link: mass 0.080 -> 0.100; geometry collision mesh filename=../meshes/IP4M_1041_pan_collision.stl; visual mesh filename=../meshes/IP4M_1041_pan_visual.obj
Joints:
- added joint amcrest_camera_frame_joint: type fixed, parent amcrest_tilt_link, child amcrest_camera_frame, origin xyz=0.035 0 0 rpy=0 0 0
- joint amcrest_camera_optical_joint: origin xyz=0.0409 0 0.006 rpy=-1.57079632679 0 -1.57079632679 -> xyz=0 0 0 rpy=-1.57079632679 0 -1.57079632679; parent amcrest_camera_link -> amcrest_camera_frame
- joint amcrest_pan_joint: limit (none) -> effort=1.0 velocity=2.5; origin xyz=0 0 0.026 rpy=0 0 0 -> xyz=0 0 0.036 rpy=0 0 0
- joint amcrest_tilt_joint: child amcrest_camera_link -> amcrest_tilt_link; limit lower=-1.22173 upper=0.436332 effort=0.5 velocity=1.0 -> lower=-1.57079632679 upper=0.78539816339 effort=1.0 velocity=2.0; origin xyz=0 0 0.051 rpy=0 0 0 -> xyz=-0.000281259 0.001454012 0.044 rpy=0 0 0

Commit message: better IP4M

File: Amcrest/IP4M-1041/urdf/IP4M-1041.urdf (robot description, URDF)
Before this commit: robot amcrest_ip4m_1041b, 5 links, 4 joints
Joints:
- joint amcrest_camera_frame_joint: origin xyz=0.035 0 0 rpy=0 0 0 -> xyz=0 -0.035 0 rpy=0 0 -1.57079632679
- joint amcrest_tilt_joint: axis 0 1 0 -> 1 0 0
