Commit message: update rail bogie in order to allow for movement

File: Generic_Objects/Rail_Bogie/urdf/rail_bogie.urdf (robot description, URDF)
Before this commit: robot rail_bogie, 3 links, 2 joints
Links:
- added link rail_base_link, mass 1
- link bogie_frame_link: geometry collision mesh filename=../meshes/rail_bogie_frame_collision.stl scale=0.09 0.09 0.09; visual mesh filename=../meshes/rail_bogie_frame_visual.obj scale=0.09 0.09 0.09
- link front_wheelset_link: geometry collision mesh filename=../meshes/rail_bogie_front_wheelset_collision.stl scale=0.09 0.09 0.09; visual mesh filename=../meshes/rail_bogie_front_wheelset_visual.obj scale=0.09 0.09 0.09
- link rear_wheelset_link: geometry collision mesh filename=../meshes/rail_bogie_rear_wheelset_collision.stl scale=0.09 0.09 0.09; visual mesh filename=../meshes/rail_bogie_rear_wheelset_visual.obj scale=0.09 0.09 0.09
Joints:
- added joint rail_joint: type prismatic, parent rail_base_link, child bogie_frame_link, origin xyz=0 0 0 rpy=0 0 0, axis 1 0 0, limit lower=-100 upper=100 effort=20000 velocity=2
- joint front_wheelset_joint: origin xyz=-3.403616428 0 0 rpy=0 0 0 -> xyz=-0.30632547852 0 0 rpy=0 0 0
- joint rear_wheelset_joint: origin xyz=3.403616428 0 0 rpy=0 0 0 -> xyz=0.30632547852 0 0 rpy=0 0 0
