Commit message: Update mesh file path in realsense_l515.urdf

File: intel/realsenseL515/urdf/realsense_l515.urdf (robot description, URDF)
Before this commit: robot realsense_l515, 1 links, 0 joints
Links:
- link realsense_l515_link: geometry collision cylinder length=0.026 radius=0.0305; visual mesh filename=../../meshes/l515.dae

Commit message: Update mesh filename path in realsense_l515.urdf

File: intel/realsenseL515/urdf/realsense_l515.urdf (robot description, URDF)
Before this commit: robot realsense_l515, 1 links, 0 joints
Links:
- link realsense_l515_link: geometry collision cylinder length=0.026 radius=0.0305; visual mesh filename=package://realsense/meshes/l515.dae
