Commit message: Update Kinova Gen3 6DoF vision URDFs
Co-Authored-By: Claude Sonnet 5.5 <noreply@anthropic.com>

File: Kinova/kinova-robotics/kortex-gen3-6dof-vision-robotiq2f85/urdf/kinova_gen3_6dof_vision_robotiq2f85.urdf (robot description, URDF)
Before this commit: robot gen3, 21 links, 20 joints
Links:
- link base_link: geometry collision mesh filename=../kortex_description/arms/gen3/6dof/meshes/base_link.STL; visual mesh filename=../kortex_description/arms/gen3/6dof/meshes/base_link.STL
- link bicep_link: geometry collision mesh filename=../kortex_description/arms/gen3/6dof/meshes/bicep_link.STL; visual mesh filename=../kortex_description/arms/gen3/6dof/meshes/bicep_link.STL
- link bracelet_link: geometry collision mesh filename=../kortex_description/arms/gen3/6dof/meshes/bracelet_with_v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; visual mesh filename=../kortex_description/arms/gen3/6dof/meshes/bracelet_with_v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
- link forearm_link: geometry collision mesh filename=../kortex_description/arms/gen3/6dof/meshes/forearm_link.STL; visual mesh filename=../kortex_description/arms/gen3/6dof/meshes/forearm_link.STL
- link robotiq_85_base_link: geometry collision mesh filename=../robotiq_description/meshes/collision/2f_85/robotiq_base.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; visual mesh filename=../robotiq_description/meshes/visual/2f_85/robotiq_base.dae
- link robotiq_85_left_finger_link: geometry collision mesh filename=../robotiq_description/meshes/collision/2f_85/left_finger.s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; visual mesh filename=../robotiq_description/meshes/visual/2f_85/left_finger.dae
- link robotiq_85_left_finger_tip_link: geometry collision mesh filename=../robotiq_description/meshes/collision/2f_85/left_finger_t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; visual mesh filename=../robotiq_description/meshes/visual/2f_85/left_finger_tip.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
- link robotiq_85_left_inner_knuckle_link: geometry collision mesh filename=../robotiq_description/meshes/collision/2f_85/left_inner_kn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; visual mesh filename=../robotiq_description/meshes/visual/2f_85/left_inner_knuck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
- link robotiq_85_left_knuckle_link: geometry collision mesh filename=../robotiq_description/meshes/collision/2f_85/left_knuckle.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; visual mesh filename=../robotiq_description/meshes/visual/2f_85/left_knuckle.dae
- link robotiq_85_right_finger_link: geometry collision mesh filename=../robotiq_description/meshes/collision/2f_85/right_finger.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; visual mesh filename=../robotiq_description/meshes/visual/2f_85/right_finger.dae
- link robotiq_85_right_finger_tip_link: geometry collision mesh filename=../robotiq_description/meshes/collision/2f_85/right_finger_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; visual mesh filename=../robotiq_description/meshes/visual/2f_85/right_finger_tip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
- link robotiq_85_right_inner_knuckle_link: geometry collision mesh filename=../robotiq_description/meshes/collision/2f_85/right_inner_k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; visual mesh filename=../robotiq_description/meshes/visual/2f_85/right_inner_knuc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
- link robotiq_85_right_knuckle_link: geometry collision mesh filename=../robotiq_description/meshes/collision/2f_85/right_knuckle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; visual mesh filename=../robotiq_description/meshes/visual/2f_85/right_knuckle.dae
- link shoulder_link: geometry collision mesh filename=../kortex_description/arms/gen3/6dof/meshes/shoulder_link.S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; visual mesh filename=../kortex_description/arms/gen3/6dof/meshes/shoulder_link.S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
- link spherical_wrist_1_link: geometry collision mesh filename=../kortex_description/arms/gen3/6dof/meshes/spherical_wrist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; visual mesh filename=../kortex_description/arms/gen3/6dof/meshes/spherical_wrist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
- link spherical_wrist_2_link: geometry collision mesh filename=../kortex_description/arms/gen3/6dof/meshes/spherical_wrist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; visual mesh filename=../kortex_description/arms/gen3/6dof/meshes/spherical_wrist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

File: Kinova/kinova-robotics/kortex-gen3-6dof-vision/urdf/kinova_gen3_6dof_vision.urdf (robot description, URDF)
Before this commit: robot gen3, 13 links, 12 joints
Links:
- link base_link: geometry collision mesh filename=../kortex_description/arms/gen3/6dof/meshes/base_link.STL; visual mesh filename=../kortex_description/arms/gen3/6dof/meshes/base_link.STL
- link bicep_link: geometry collision mesh filename=../kortex_description/arms/gen3/6dof/meshes/bicep_link.STL; visual mesh filename=../kortex_description/arms/gen3/6dof/meshes/bicep_link.STL
- link bracelet_link: geometry collision mesh filename=../kortex_description/arms/gen3/6dof/meshes/bracelet_with_v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; visual mesh filename=../kortex_description/arms/gen3/6dof/meshes/bracelet_with_v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
- link forearm_link: geometry collision mesh filename=../kortex_description/arms/gen3/6dof/meshes/forearm_link.STL; visual mesh filename=../kortex_description/arms/gen3/6dof/meshes/forearm_link.STL
- link shoulder_link: geometry collision mesh filename=../kortex_description/arms/gen3/6dof/meshes/shoulder_link.S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; visual mesh filename=../kortex_description/arms/gen3/6dof/meshes/shoulder_link.S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
- link spherical_wrist_1_link: geometry collision mesh filename=../kortex_description/arms/gen3/6dof/meshes/spherical_wrist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; visual mesh filename=../kortex_description/arms/gen3/6dof/meshes/spherical_wrist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
- link spherical_wrist_2_link: geometry collision mesh filename=../kortex_description/arms/gen3/6dof/meshes/spherical_wrist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; visual mesh filename=../kortex_description/arms/gen3/6dof/meshes/spherical_wrist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
